File: tests/fixtures/kicad/features.kicad_pcb (KiCad board)
At the start: 20 x 10 mm, 5 parts, among them J1 front, J2 back

Commit message: feat(core): add semantic port_cutout (#29)
* test(core): specify semantic port cutouts

* feat(core): add semantic port cutouts

* test(core): update port cutout kind contracts

* test(core): cover enclosure modifier conflicts

* fix(core): compose enclosure modifiers by base

* test(core): cover unified body modifier lineage

* fix(core): unify body modifier lineage

* deslop(core): remove legacy port target loader

* refactor(core): isolate port opening bounds

* chore(core): sort lineage test imports

* refactor(core): trust lineage terminal catalog

* fix(mcp): keep BODY_LINEAGE_DIVERGED as its own error code
Parts:
- added J3: center, Connector:Center, F.Cu at (10.0, 5.00)
- moved J1 3.00 mm to (1.00, 5.00), turned to 0 degrees
Changed lines of the file:
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@@
   (property "Reference" "H1") (property "Value" "NPTH")
   (pad "" np_thru_hole circle (at 0 0) (drill 1.5) (layers "*.Cu" "*.Mask")))
- (footprint "Connector:Front" (layer "F.Cu") (uuid "front-id") (at 4 5 45)
+ (footprint "Connector:Front" (layer "F.Cu") (uuid "front-id") (at 1 5)
   (property "Reference" "J1") (property "Value" "front")
+  (fp_rect (start -1 -2) (end 1 2) (stroke (width 0.05) (type default))
+   (fill none) (layer "F.CrtYd"))
   (model "${KICAD8_3DMODEL_DIR}/front.wrl"))
+ (footprint "Connector:Center" (layer "F.Cu") (uuid "center-id") (at 10 5)
+  (property "Reference" "J3") (property "Value" "center"))
  (footprint "Connector:Back" (layer "B.Cu") (uuid "back-id") (at 16 5 270)
   (property "Reference" "J2") (property "Value" "back")
