File: evals/fixtures/features-moved.kicad_pcb (KiCad board)
At the start: 20 x 10 mm, 6 parts, among them J1 front, J2 back, J3 center

Commit message: fix(evals): prove refreshed board movement
Parts:
- moved J1 2.00 mm to (3.00, 5.00)
Changed lines of the file:
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@@
   (property "Reference" "H1") (property "Value" "NPTH")
   (pad "" np_thru_hole circle (at 0 0) (drill 1.5) (layers "*.Cu" "*.Mask")))
- (footprint "Connector:Front" (layer "F.Cu") (uuid "front-id") (at 1 5)
+ (footprint "Connector:Front" (layer "F.Cu") (uuid "front-id") (at 3 5)
   (property "Reference" "J1") (property "Value" "front")
   (fp_rect (start -1 -2) (end 1 2) (stroke (width 0.05) (type default))
